File: 8Q/qpu.sch (KiCad schematic (older format))
At the start: 232 parts

Commit message: modified:   8Q/8Q-cache.lib 	modified:   8Q/8Q.sch 	modified:   8Q/8_qp_io.sch 	new file:   8Q/RAM.sch 	deleted:    8Q/_saved_RAM.sch 	modified:   8Q/cpu.sch 	modified:   8Q/cpu_power.sch 	modified:   8Q/power.sch 	modified:   8Q/preprocessor.sch 	modified:   8Q/qpower.sch 	modified:   8Q/qpu.sch 	new file:   8q.dia 	modified:   README.md 	new file:   docs/source/imgs/8q.png
Connections:
- net at M?.~ (V): now also U?.~ (Oin); no longer U?.~ (Oin) (x8)
- net at U?.~ (Oin): now also U?.~ (Oin); no longer M?.~ (V) (x7)
- net at U?.~ (Oin): now also U?.~ (Oin); no longer U?.~ (Vcc) (x7)
- net at U?.~ (Oin): now also U?.~ (S5); no longer U?.~ (S5) (x2)
- net at U?.~ (Oin): now also U?.~ (S5); no longer U?.~ (Oin) (x20)
- net at U?.~ (S5): no longer U?.~ (Oin) (x2)
- net at U?.~ (S5): now also U?.~ (Oin); no longer U?.~ (Oin) (x10)
- net at U?.~ (Oin): now also U?.~ (S2); no longer U?.~ (S5) (x2)
- net at U?.~ (S2): now also U?.~ (S2); no longer U?.~ (Oin) (x2)
- net at U?.~ (Oin): now also U?.~ (Oin); no longer U?.~ (S5) (x16)
- net at U?.~ (S5): now also H?.3 (Vout); no longer U?.~ (Oin) (x2)
- net at U?.~ (S5): now also H?.4 (Hout); no longer U?.~ (Oin) (x2)
- net at U?.~ (S2): now also U?.~ (Oin); no longer U?.~ (Oin) (x9)
- net at U?.~ (Oin): now also U?.~ (Vcc); no longer U?.~ (Oin) (x2)
- net at U?.~ (S2): now also U?.~ (Vcc); no longer U?.~ (S2) (x7)
- net at U?.~ (S2): now also U?.~ (Oin); no longer U?.~ (Vcc) (x4)
- net at U?.~ (Oin): now also U?.~ (S5); no longer U?.~ (S2) (x4)
- net at U?.~ (S2): now also SPE?.5 (V); no longer U?.~ (S2) (x2)
- net at U?.~ (S2): now also SPE?.4 (H); no longer U?.~ (S2) (x2)
- new net: M?.~ (V), U?.~ (Oin) (x8)
- new net: U?.~ (Oin), U?.~ (Vcc) (x18)
- new net: U?.~ (Vcc), U?.~ (Vcc) (x9)
- new net: U?.~ (Oin), U?.~ (S5) (x16)
- new net: U?.~ (Oin), U?.~ (Oin) (x22)
- new net: U?.~ (Oin), U?.~ (S2) (x16)
- new net: U?.~ (S2), U?.~ (Vcc) (x8)
- new net: U?.~ (S2), U?.~ (S2) (x10)
- new net: U?.~ (S5), U?.~ (Vcc) (x4)
- now unconnected: U?.~ (S5), U?.~ (S5), U?.~ (S5), U?.~ (S5)
Changed lines of the file:
@@
 $Descr User 47992 35433
 encoding utf-8
-Sheet 4 8
+Sheet 5 9
 Title "8Q Quantum Computer"
 Date "2020-06-29"

Commit message: modified:   8Q/8Q-cache.lib 	modified:   8Q/8Q.sch 	modified:   8Q/8_qp_io.sch 	modified:   8Q/RAM.sch 	new file:   8Q/control_logic.sch 	modified:   8Q/cpu.sch 	modified:   8Q/cpu_power.sch 	new file:   8Q/inorder.sch 	new file:   8Q/instruction_bus.sch 	new file:   8Q/output_cache.sch 	modified:   8Q/power.sch 	modified:   8Q/preprocessor.sch 	modified:   8Q/qpower.sch 	modified:   8Q/qpu.sch 	new file:   Controller.md 	modified:   QCore.md 	new file:   QPU_Operation.md 	new file:   docs/source/imgs/Screenshot from 2020-07-07 18-04-51.png 	new file:   tools/photon_birth_death.py 	new file:   tools/processor.py
Parts:
- removed U? (x7): HEF4093B, symbol 4xxx:HEF4093B
- added U175: HEF4093B, Package_DIP:DIP-14_W7.62mm, symbol 4xxx:HEF4093B
- added unit 2 of U176
- added unit 4 of U176
- added unit 3 of U176
- CH1: renamed from CH?; footprint (none) -> Quantum:Macro-CZX-Gate
- CX1: renamed from CX?; footprint (none) -> Quantum:Macro-CX-Gate
- CY1: renamed from CY?; footprint (none) -> Quantum:Macro-CY-Gate
- CZ1: renamed from CZ?; footprint (none) -> Quantum:Macro-CZ-Gate
- H1, H2, H3, H4, H5, H6, H7, H8: renamed from H?; footprint (none) -> Quantum:Macro-X-Gate
- M1, M2, M3, M4, M5, M6, M7: renamed from M?; footprint (none) -> Quantum:Macro-Measure
- M8: renamed from M?; footprint (none) -> Quantum:Macro-Photon-Source
- SPE1, SPE2, SPE3, SPE4, SPE5, SPE6, SPE7, SPE8: renamed from SPE?; footprint (none) -> Quantum:Macro-Photon-Source
- U176: renamed from U?; footprint (none) -> Package_DIP:DIP-14_W7.62mm
- X1, X2, X3, X4, X5, X6, X7, X8: renamed from X?; footprint (none) -> Quantum:Macro-X-Gate
- Y1, Y2, Y3, Y4, Y5, Y6, Y7, Y8: renamed from Y?; footprint (none) -> Quantum:Macro-Y-Gate
- Z1, Z2, Z3, Z4, Z5, Z6, Z7, Z8: renamed from Z?; footprint (none) -> Quantum:Macro-X-Gate
- gave numbers to parts that had none: 172
Connections:
- net CQ1 is gone; now on net Q3Z: U173.~ (Vcc), U174.~ (Vcc)
- net CQ2 is gone; now on net Q3Z: U173.~ (Vcc), U174.~ (Vcc)
- net CQ3 is gone; now on net Q3Z: U173.~ (Vcc), U174.~ (Vcc)
- net Q2-Out: now also U176.6
- net Q2-S: now also U176.4
- net Q3-Out: now also U175.9
- net Q3-S: now also U175.10
- net Q4-Out: now also U176.13
- net Q4-S: now also U176.11
- net Q5-Out: now also U175.2
- net Q5-S: now also U175.3
- net Q6-Out: now also U175.6
- net Q6-S: now also U175.4
- net Q7-Out: now also U176.9
- net Q7-S: now also U176.10
- net Q8-Out: now also U175.13
- net Q8-S: now also U175.11
- net at M8.~ (V): now also U38.~ (Oin); no longer U37.~ (Oin)
- net at U38.~ (Oin): now also U58.~ (Oin); no longer M8.~ (V)
- net at U37.~ (Oin): now also U57.~ (Oin); no longer U25.~ (Vcc)
- net at U40.~ (Oin): now also U82.~ (S5); no longer U28.~ (S5)
- net at U34.~ (Oin): now also U28.~ (S5); no longer U40.~ (Oin)
- net at U82.~ (S5): no longer U40.~ (Oin)
- net at U45.~ (Oin): now also U43.~ (S5); no longer U53.~ (Oin)
- net at U43.~ (S5): now also U53.~ (Oin); no longer U45.~ (Oin)
- net at U53.~ (Oin): now also U83.~ (S5); no longer U43.~ (S5)
- net at U83.~ (S5): no longer U53.~ (Oin)
- net at U74.~ (Oin): now also U87.~ (S2); no longer U56.~ (S5)
- net at U68.~ (Oin): now also U56.~ (S5); no longer U74.~ (Oin)
- net at U87.~ (S2): now also U103.~ (S2); no longer U74.~ (Oin)
- net at U85.~ (Oin): now also U77.~ (S5); no longer U91.~ (Oin)
- net at U77.~ (S5): now also U91.~ (Oin); no longer U85.~ (Oin)
- net at U91.~ (Oin): now also U89.~ (S2); no longer U77.~ (S5)
- net at U89.~ (S2): now also U104.~ (S2); no longer U91.~ (Oin)
- net at U106.~ (Oin): now also U112.~ (Oin); no longer U96.~ (S5)
- net at U102.~ (Oin): now also U96.~ (S5); no longer U106.~ (Oin)
- net at U96.~ (S5): now also H4.3 (Vout); no longer U102.~ (Oin)
- net at U118.~ (Oin): now also U114.~ (S5); no longer U124.~ (Oin)
- net at U114.~ (S5): now also H4.4 (Hout); no longer U118.~ (Oin)
- net at U124.~ (Oin): now also U126.~ (Oin); no longer U114.~ (S5)
- net at U116.~ (S2): now also U65.~ (Oin); no longer U112.~ (Oin)
- net at U122.~ (S2): now also U66.~ (Oin); no longer U126.~ (Oin)
- net at U136.~ (Oin): now also U141.~ (Oin); no longer U128.~ (S5)
- net at U130.~ (Oin): now also U128.~ (S5); no longer U136.~ (Oin)
- net at U146.~ (Oin): now also U144.~ (S5); no longer U148.~ (Oin)
- net at U144.~ (S5): now also U148.~ (Oin); no longer U146.~ (Oin)
- net at U148.~ (Oin): now also U152.~ (Oin); no longer U144.~ (S5)
- net at U134.~ (S2): now also U69.~ (Oin); no longer U141.~ (Oin)
- net at U160.~ (Oin): now also U162.~ (Oin); no longer U154.~ (S5)
- net at U158.~ (Oin): now also U154.~ (S5); no longer U160.~ (Oin)
- net at U166.~ (Oin): now also U164.~ (S5); no longer U168.~ (Oin)
- net at U164.~ (S5): now also U168.~ (Oin); no longer U166.~ (Oin)
- net at U168.~ (Oin): now also U170.~ (Oin); no longer U164.~ (S5)
- net at U31.~ (Oin): now also U17.~ (Vcc); no longer U63.~ (Oin)
- net at U32.~ (Oin): now also U18.~ (Vcc); no longer U64.~ (Oin)
- net at M6.1 (Hd): now also U176.5
- net at M6.~ (V): now also U32.~ (Oin); no longer U31.~ (Oin)
- net at M4.1 (Hd): now also U175.8
- net at M4.~ (V): now also U22.~ (Oin); no longer U21.~ (Oin)
- net at U22.~ (Oin): now also U66.~ (Oin); no longer M4.~ (V)
- net at U21.~ (Oin): now also U65.~ (Oin); no longer U9.~ (Vcc)
- net at M2.1 (Hd): now also U176.12
- net at M2.~ (V): now also U14.~ (Oin); no longer U13.~ (Oin)
- net at U14.~ (Oin): now also U70.~ (Oin); no longer M2.~ (V)
- net at U13.~ (Oin): now also U69.~ (Oin); no longer U5.~ (Vcc)
- net at U104.~ (S2): now also U174.~ (Vcc); no longer U89.~ (S2)
- net at U103.~ (S2): now also U173.~ (Vcc); no longer U87.~ (S2)
- net at U78.~ (S2): now also U99.~ (Oin); no longer U59.~ (Vcc)
- net at U79.~ (S2): now also U100.~ (Oin); no longer U60.~ (Vcc)
- net at U80.~ (S2): now also U98.~ (Oin); no longer U61.~ (Vcc)
- net at U81.~ (S2): now also U99.~ (Oin); no longer U62.~ (Vcc)
- net at U132.~ (S2): now also U174.~ (Vcc); no longer U122.~ (S2)
- net at U131.~ (S2): now also U173.~ (Vcc); no longer U116.~ (S2)
- net at U97.~ (Oin): now also U107.~ (S5); no longer U78.~ (S2)
- net at U149.~ (S2): now also U173.~ (Vcc); no longer U134.~ (S2)
- net at U98.~ (Oin): now also U108.~ (S5); no longer U79.~ (S2)
- net at U100.~ (Oin): now also U110.~ (S5); no longer U79.~ (S2)
- net at U99.~ (Oin): now also U109.~ (S5); no longer U78.~ (S2)
- net at U156.~ (S2): now also U172.~ (Vcc); no longer U133.~ (S2)
- net at U155.~ (S2): now also U171.~ (Vcc); no longer U137.~ (S2)
- net at M7.2 (Vd): now also U175.12
- net at M7.~ (V): now also U35.~ (Oin); no longer U36.~ (Oin)
- net at U35.~ (Oin): now also U71.~ (Oin); no longer M7.~ (V)
- net at U36.~ (Oin): now also U72.~ (Oin); no longer U24.~ (Vcc)
- net at U39.~ (Oin): now also U41.~ (Oin); no longer U27.~ (S5)
- net at U33.~ (Oin): now also U27.~ (S5); no longer U39.~ (Oin)
- net at U44.~ (Oin): now also U42.~ (S5); no longer U52.~ (Oin)
- net at U42.~ (S5): now also U52.~ (Oin); no longer U44.~ (Oin)
- net at U52.~ (Oin): now also U54.~ (Oin); no longer U42.~ (S5)
- net at U73.~ (Oin): now also U75.~ (Oin); no longer U55.~ (S5)
- net at U67.~ (Oin): now also U55.~ (S5); no longer U73.~ (Oin)
- net at U84.~ (Oin): now also U76.~ (S5); no longer U90.~ (Oin)
- net at U76.~ (S5): now also U90.~ (Oin); no longer U84.~ (Oin)
- net at U90.~ (Oin): now also U92.~ (Oin); no longer U76.~ (S5)
- net at U105.~ (Oin): now also U111.~ (Oin); no longer U95.~ (S5)
- net at U101.~ (Oin): now also U95.~ (S5); no longer U105.~ (Oin)
- net at U95.~ (S5): now also H3.3 (Vout); no longer U101.~ (Oin)
- net at U117.~ (Oin): now also U113.~ (S5); no longer U123.~ (Oin)
- net at U113.~ (S5): now also H3.4 (Hout); no longer U117.~ (Oin)
- net at U123.~ (Oin): now also U125.~ (Oin); no longer U113.~ (S5)
- net at U93.~ (S5): now also U71.~ (Oin); no longer U54.~ (Oin)
- net at U94.~ (S5): now also U72.~ (Oin); no longer U41.~ (Oin)
- net at U86.~ (S2): now also U51.~ (Oin); no longer U75.~ (Oin)
- net at U88.~ (S2): now also U50.~ (Oin); no longer U92.~ (Oin)
- net at U115.~ (S2): now also U49.~ (Oin); no longer U111.~ (Oin)
- net at U121.~ (S2): now also U48.~ (Oin); no longer U125.~ (Oin)
- net at U135.~ (Oin): now also U140.~ (Oin); no longer U127.~ (S5)
- net at U129.~ (Oin): now also U127.~ (S5); no longer U135.~ (Oin)
- net at U145.~ (Oin): now also U143.~ (S5); no longer U147.~ (Oin)
- net at U143.~ (S5): now also U147.~ (Oin); no longer U145.~ (Oin)
- net at U147.~ (Oin): now also U151.~ (Oin); no longer U143.~ (S5)
- net at U133.~ (S2): now also U47.~ (Oin); no longer U140.~ (Oin)
- net at U137.~ (S2): now also U46.~ (Oin); no longer U151.~ (Oin)
- net at U159.~ (Oin): now also U161.~ (Oin); no longer U153.~ (S5)
- net at U157.~ (Oin): now also U153.~ (S5); no longer U159.~ (Oin)
- net at U165.~ (Oin): now also U163.~ (S5); no longer U167.~ (Oin)
- net at U163.~ (S5): now also U167.~ (Oin); no longer U165.~ (Oin)
- net at U167.~ (Oin): now also U169.~ (Oin); no longer U163.~ (S5)
- net at M5.2 (Vd): now also U176.8
- net at M5.~ (V): now also U29.~ (Oin); no longer U30.~ (Oin)
- net at U29.~ (Oin): now also U50.~ (Oin); no longer M5.~ (V)
- net at U30.~ (Oin): now also U51.~ (Oin); no longer U16.~ (Vcc)
- net at M3.2 (Vd): now also U175.5
- net at M3.~ (V): now also U19.~ (Oin); no longer U20.~ (Oin)
- net at U19.~ (Oin): now also U48.~ (Oin); no longer M3.~ (V)
- net at U20.~ (Oin): now also U49.~ (Oin); no longer U8.~ (Vcc)
- net at M1.2 (Vd): now also U175.1
- net at M1.~ (V): now also U11.~ (Oin); no longer U12.~ (Oin)
- net at U11.~ (Oin): now also U46.~ (Oin); no longer M1.~ (V)
- net at U12.~ (Oin): now also U47.~ (Oin); no longer U4.~ (Vcc)
- net at U119.~ (S2): now also SPE4.5 (V); no longer U88.~ (S2)
- net at U120.~ (S2): now also SPE4.4 (H); no longer U86.~ (S2)
- net at U138.~ (S2): now also SPE6.5 (V); no longer U121.~ (S2)
- net at U139.~ (S2): now also SPE6.4 (H); no longer U115.~ (S2)
- new net: M8.~ (V), U37.~ (Oin)
- new net: U25.~ (Vcc), U37.~ (Oin)
- new net: U25.~ (Vcc), U26.~ (Vcc)
- new net: U26.~ (Vcc), U38.~ (Oin)
- new net: U28.~ (S5), U40.~ (Oin)
- new net: U34.~ (Oin), U40.~ (Oin)
- new net: U45.~ (Oin), U53.~ (Oin)
- new net: U56.~ (S5), U74.~ (Oin)
- new net: U68.~ (Oin), U74.~ (Oin)
- new net: U85.~ (Oin), U91.~ (Oin)
- new net: U106.~ (Oin), U96.~ (S5)
- new net: U102.~ (Oin), U106.~ (Oin)
- new net: U118.~ (Oin), U124.~ (Oin)
- new net: U114.~ (S5), U124.~ (Oin)
- new net: U112.~ (Oin), U116.~ (S2)
- new net: U122.~ (S2), U126.~ (Oin)
- new net: U128.~ (S5), U136.~ (Oin)
- new net: U130.~ (Oin), U136.~ (Oin)
- new net: U146.~ (Oin), U148.~ (Oin)
- new net: U134.~ (S2), U141.~ (Oin)
- new net: U154.~ (S5), U160.~ (Oin)
- new net: U158.~ (Oin), U160.~ (Oin)
- new net: U166.~ (Oin), U168.~ (Oin)
- new net: U162.~ (Oin), U173.~ (Vcc)
- new net: U170.~ (Oin), U174.~ (Vcc)
- new net: U31.~ (Oin), U63.~ (Oin)
- new net: U63.~ (Oin), U87.~ (S2)
- new net: U32.~ (Oin), U64.~ (Oin)
- new net: U64.~ (Oin), U89.~ (S2)
- new net: M6.~ (V), U31.~ (Oin)
- new net: U17.~ (Vcc), U18.~ (Vcc)
- new net: M4.~ (V), U21.~ (Oin)
- new net: U21.~ (Oin), U9.~ (Vcc)
- new net: U10.~ (Vcc), U9.~ (Vcc)
- new net: U10.~ (Vcc), U22.~ (Oin)
- new net: M2.~ (V), U13.~ (Oin)
- new net: U13.~ (Oin), U5.~ (Vcc)
- new net: U5.~ (Vcc), U6.~ (Vcc)
- new net: U14.~ (Oin), U6.~ (Vcc)
- new net: U59.~ (Vcc), U78.~ (S2)
- new net: U60.~ (Vcc), U79.~ (S2)
- new net: U61.~ (Vcc), U80.~ (S2)
- new net: U62.~ (Vcc), U81.~ (S2)
- new net: U122.~ (S2), U132.~ (S2)
- new net: U116.~ (S2), U131.~ (S2)
- new net: U78.~ (S2), U97.~ (Oin)
- new net: U80.~ (S2), U97.~ (Oin)
- new net: U142.~ (S2), U150.~ (S2)
- new net: U134.~ (S2), U149.~ (S2)
- new net: U79.~ (S2), U98.~ (Oin)
- new net: U100.~ (Oin), U81.~ (S2)
- new net: U142.~ (S2), U70.~ (Oin)
- new net: U173.~ (Vcc), U82.~ (S5)
- new net: U174.~ (Vcc), U83.~ (S5)
- new net: U133.~ (S2), U156.~ (S2)
- new net: U137.~ (S2), U155.~ (S2)
- new net: M7.~ (V), U36.~ (Oin)
- new net: U24.~ (Vcc), U36.~ (Oin)
- new net: U23.~ (Vcc), U24.~ (Vcc)
- new net: U23.~ (Vcc), U35.~ (Oin)
- new net: U27.~ (S5), U39.~ (Oin)
- new net: U33.~ (Oin), U39.~ (Oin)
- new net: U44.~ (Oin), U52.~ (Oin)
- new net: U55.~ (S5), U73.~ (Oin)
- new net: U67.~ (Oin), U73.~ (Oin)
- new net: U84.~ (Oin), U90.~ (Oin)
- new net: U105.~ (Oin), U95.~ (S5)
- new net: U101.~ (Oin), U105.~ (Oin)
- new net: U117.~ (Oin), U123.~ (Oin)
- new net: U113.~ (S5), U123.~ (Oin)
- new net: U54.~ (Oin), U93.~ (S5)
- new net: U41.~ (Oin), U94.~ (S5)
- new net: U75.~ (Oin), U86.~ (S2)
- new net: U88.~ (S2), U92.~ (Oin)
- new net: U111.~ (Oin), U115.~ (S2)
- new net: U121.~ (S2), U125.~ (Oin)
- new net: U127.~ (S5), U135.~ (Oin)
- new net: U129.~ (Oin), U135.~ (Oin)
- new net: U145.~ (Oin), U147.~ (Oin)
- new net: U133.~ (S2), U140.~ (Oin)
- new net: U137.~ (S2), U151.~ (Oin)
- new net: U153.~ (S5), U159.~ (Oin)
- new net: U157.~ (Oin), U159.~ (Oin)
- new net: U165.~ (Oin), U167.~ (Oin)
- new net: U161.~ (Oin), U172.~ (Vcc)
- new net: U169.~ (Oin), U171.~ (Vcc)
- new net: M5.~ (V), U30.~ (Oin)
- new net: U16.~ (Vcc), U30.~ (Oin)
- new net: U15.~ (Vcc), U16.~ (Vcc)
- new net: U15.~ (Vcc), U29.~ (Oin)
- new net: M3.~ (V), U20.~ (Oin)
- new net: U20.~ (Oin), U8.~ (Vcc)
- new net: U7.~ (Vcc), U8.~ (Vcc)
- new net: U19.~ (Oin), U7.~ (Vcc)
- new net: M1.~ (V), U12.~ (Oin)
- new net: U12.~ (Oin), U4.~ (Vcc)
- new net: U3.~ (Vcc), U4.~ (Vcc)
- new net: U11.~ (Oin), U3.~ (Vcc)
- new net: U119.~ (S2), U88.~ (S2)
- new net: U120.~ (S2), U86.~ (S2)
- new net: U121.~ (S2), U138.~ (S2)
- new net: U115.~ (S2), U139.~ (S2)
- new net: U171.~ (Vcc), U172.~ (Vcc)
- new net: U139.~ (S2), U172.~ (Vcc)
- new net: U120.~ (S2), U172.~ (Vcc)
- new net: U172.~ (Vcc), U94.~ (S5)
- new net: U138.~ (S2), U171.~ (Vcc)
- new net: U119.~ (S2), U171.~ (Vcc)
- new net: U171.~ (Vcc), U93.~ (S5)
- new net: U57.~ (Oin), U82.~ (S5)
- new net: U58.~ (Oin), U83.~ (S5)
- new net CQ1D: U173.~ (Vcc), U174.~ (Vcc)
- new net CQ2D: U173.~ (Vcc), U174.~ (Vcc)
- new net CQ3D: U173.~ (Vcc), U174.~ (Vcc)
- now unconnected: U82.~ (S5), U82.~ (S5), U83.~ (S5), U83.~ (S5)

Commit message: modified:   8Q/8Q-cache.lib 	new file:   8Q/8Q-rescue.dcm 	new file:   8Q/8Q-rescue.lib 	modified:   8Q/8Q.kicad_pcb 	modified:   8Q/8Q.sch 	modified:   8Q/8_qp_io.sch 	new file:   8Q/QGates.pretty/CH-Gate.kicad_mod 	new file:   8Q/QGates.pretty/CX-Gate.kicad_mod 	new file:   8Q/QGates.pretty/CY-Gate.kicad_mod 	new file:   8Q/QGates.pretty/CZ-Gate.kicad_mod 	new file:   8Q/QGates.pretty/H-Gate.kicad_mod 	new file:   8Q/QGates.pretty/Measure.kicad_mod 	new file:   8Q/QGates.pretty/Photon-Source.kicad_mod 	new file:   8Q/QGates.pretty/X-Gate.kicad_mod 	new file:   8Q/QGates.pretty/Y-Gate.kicad_mod 	new file:   8Q/QGates.pretty/Z-Gate.kicad_mod 	modified:   8Q/control_logic.sch 	modified:   8Q/cpu.sch 	modified:   8Q/inorder.sch 	modified:   8Q/instruction_bus.sch 	modified:   8Q/output_cache.sch 	modified:   8Q/power.sch 	modified:   8Q/preprocessor.sch 	modified:   8Q/qpower.sch 	modified:   8Q/qpu.sch 	new file:   8Q/sym-lib-table Introduced embedded QSeven module to replace CPU Computer now has support for: * 10Gbps Ethernet * 1xUSB3.0 * 4xUSB2.0 * 1xJTAG * 1xCAN * 1-Wire Bus * 1xSMBus * 1xI2C * External Watchdog * HDMI * LVDS
Parts:
- CH1: footprint Quantum:Macro-CZX-Gate -> QGates:CH-Gate; symbol Quantum:Macro-CX-Gate -> 8Q-rescue:Macro-CX-Gate-Quantum
- CX1: footprint Quantum:Macro-CX-Gate -> QGates:CX-Gate; symbol Quantum:Macro-CX-Gate -> 8Q-rescue:Macro-CX-Gate-Quantum
- CY1: footprint Quantum:Macro-CY-Gate -> QGates:CY-Gate; symbol Quantum:Macro-CX-Gate -> 8Q-rescue:Macro-CX-Gate-Quantum
- CZ1: footprint Quantum:Macro-CZ-Gate -> QGates:CZ-Gate; symbol Quantum:Macro-CX-Gate -> 8Q-rescue:Macro-CX-Gate-Quantum
- H1, H2, H3, H4, H5, H6, H7, H8: footprint Quantum:Macro-X-Gate -> QGates:H-Gate; symbol Quantum:Macro-X-Gate -> 8Q-rescue:Macro-X-Gate-Quantum
- M1, M2, M3, M4, M5, M6, M7: footprint Quantum:Macro-Measure -> QGates:Measure; symbol Quantum:Macro-Measure -> 8Q-rescue:Macro-Measure-Quantum
- M8: footprint Quantum:Macro-Photon-Source -> QGates:Measure; symbol Quantum:Macro-Measure -> 8Q-rescue:Macro-Measure-Quantum
- SPE1, SPE2, SPE3, SPE4, SPE5, SPE6, SPE7, SPE8: footprint Quantum:Macro-Photon-Source -> QGates:Photon-Source; symbol Quantum:Macro-Photon-Source -> 8Q-rescue:Macro-Photon-Source-Quantum
- U10, U15, U16, U17, U171, U172, U173, U174, U18, U23, U24, U25, U26, U3, U4, U5, U59, U6, U60, U61, U62, U7, U8, U9: symbol Quantum:Switch-1x4 -> 8Q-rescue:Switch-1x4-Quantum
- U100, U105, U106, U11, U111, U112, U12, U123, U124, U125, U126, U13, U135, U136, U14, U140, U141, U147, U148, U151, U152, U159, U160, U161, U162, U167, U168, U169, U170, U19, U20, U21, U22, U29, U30, U31, U32, U35, U36, U37, U38, U39, U40, U41, U46, U47, U48, U49, U50, U51, U52, U53, U54, U57, U58, U63, U64, U65, U66, U69, U70, U71, U72, U73, U74, U75, U90, U91, U92, U97, U98, U99: symbol Quantum:Switch-1x2 -> 8Q-rescue:Switch-1x2-Quantum
- U101, U102, U117, U118, U129, U130, U145, U146, U157, U158, U165, U166, U33, U34, U44, U45, U67, U68, U84, U85: symbol Quantum:Delay-Loop -> 8Q-rescue:Delay-Loop-Quantum
- U103, U104, U115, U116, U119, U120, U121, U122, U131, U132, U133, U134, U137, U138, U139, U142, U149, U150, U155, U156, U78, U79, U80, U81, U86, U87, U88, U89: symbol Quantum:Collator-2x1 -> 8Q-rescue:Collator-2x1-Quantum
- U107, U108, U109, U110, U113, U114, U127, U128, U143, U144, U153, U154, U163, U164, U27, U28, U42, U43, U55, U56, U76, U77, U82, U83, U93, U94, U95, U96: symbol Quantum:Collator-5x1 -> 8Q-rescue:Collator-5x1-Quantum
- X1, X2, X3, X4, X5, X6, X7, X8: footprint Quantum:Macro-X-Gate -> QGates:X-Gate; symbol Quantum:Macro-X-Gate -> 8Q-rescue:Macro-X-Gate-Quantum
- Y1, Y2, Y3, Y4, Y5, Y6, Y7, Y8: footprint Quantum:Macro-Y-Gate -> QGates:Y-Gate; symbol Quantum:Macro-Y-Gate -> 8Q-rescue:Macro-Y-Gate-Quantum
- Z1, Z2, Z3, Z4, Z5, Z6, Z7, Z8: footprint Quantum:Macro-X-Gate -> QGates:Z-Gate; symbol Quantum:Macro-Z-Gate -> 8Q-rescue:Macro-Z-Gate-Quantum
Connections:
- net CG1H: now also U108.5 (S5); no longer U108.~ (S5)
- net CG1V: now also U107.5 (S5); no longer U107.~ (S5)
- net CG2H: now also U108.4 (S4); no longer U108.~ (S5)
- net CG2V: now also U107.4 (S4); no longer U107.~ (S5)
- net CG3H: now also U108.3 (S3), U126.5 (O1); no longer U108.~ (S5), U126.~ (Oin)
- net CG3V: now also U107.3 (S3), U112.5 (O1); no longer U107.~ (S5), U112.~ (Oin)
- net CG4H: now also U108.2 (S2), U152.5 (O1); no longer U108.~ (S5), U152.~ (Oin)
- net CG4V: now also U107.2 (S2), U141.5 (O1); no longer U107.~ (S5), U141.~ (Oin)
- net CG5H: now also U110.5 (S5), U54.5 (O1); no longer U110.~ (S5), U54.~ (Oin)
- net CG5V: now also U109.5 (S5), U41.5 (O1); no longer U109.~ (S5), U41.~ (Oin)
- net CG6H: now also U110.4 (S4), U92.5 (O1); no longer U110.~ (S5), U92.~ (Oin)
- net CG6V: now also U109.4 (S4), U75.5 (O1); no longer U109.~ (S5), U75.~ (Oin)
- net CG7H: now also U110.3 (S3), U125.5 (O1); no longer U110.~ (S5), U125.~ (Oin)
- net CG7V: now also U109.3 (S3), U111.5 (O1); no longer U109.~ (S5), U111.~ (Oin)
- net CG8H: now also U110.2 (S2), U151.5 (O1); no longer U110.~ (S5), U151.~ (Oin)
- net CG8V: now also U109.2 (S2), U140.5 (O1); no longer U109.~ (S5), U140.~ (Oin)
- net CGCH: now also U108.1 (S1), U170.5 (O1); no longer U108.~ (S5), U170.~ (Oin)
- net CGCV: now also U107.1 (S1), U162.5 (O1); no longer U107.~ (S5), U162.~ (Oin)
- net CGTH: now also U110.1 (S1), U169.5 (O1); no longer U110.~ (S5), U169.~ (Oin)
- net CGTV: now also U109.1 (S1), U161.5 (O1); no longer U109.~ (S5), U161.~ (Oin)
- net CH_TRIGGER: now also CH1.11 (S); no longer CH1.~ (Vcc)
- net CX_TRIGGER: now also CX1.11 (S); no longer CX1.~ (Vcc)
- net CY_TRIGGER: now also CY1.11 (S); no longer CY1.~ (Vcc)
- net CZ_TRIGGER: now also CZ1.11 (S); no longer CZ1.~ (Vcc)
- net GNDA: now also SPE1.7 (GND), SPE2.7 (GND), SPE3.7 (GND), SPE4.7 (GND), SPE5.7 (GND), SPE6.7 (GND), SPE7.7 (GND), SPE8.7 (GND); no longer SPE1.6 (GND), SPE2.6 (GND), SPE3.6 (GND), SPE4.6 (GND), SPE5.6 (GND), SPE6.6 (GND), SPE7.6 (GND), SPE8.6 (GND)
- net Q1H: now also U58.5 (O1); no longer U58.~ (Oin)
- net Q1SR: now also SPE1.2 (Set/Reset); no longer SPE1.~ (Set/Reset)
- net Q1V: now also U57.5 (O1); no longer U57.~ (Oin)
- net Q2H: now also U64.5 (O1); no longer U64.~ (Oin)
- net Q2SR: now also SPE3.2 (Set/Reset); no longer SPE3.~ (Set/Reset)
- net Q2V: now also U63.5 (O1); no longer U63.~ (Oin)
- net Q3H: now also U66.5 (O1); no longer U66.~ (Oin)
- net Q3SR: now also SPE5.2 (Set/Reset); no longer SPE5.~ (Set/Reset)
- net Q3T: now also U142.2 (S2), U150.1 (S1), U152.4 (O2); no longer U142.~ (S2), U150.~ (S2), U152.~ (Oin)
- net Q3V: now also U65.5 (O1); no longer U65.~ (Oin)
- net Q4H: now also U70.5 (O1); no longer U70.~ (Oin)
- net Q4SR: now also SPE7.2 (Set/Reset); no longer SPE7.~ (Set/Reset)
- net Q4V: now also U69.5 (O1); no longer U69.~ (Oin)
- net Q5H: now also U46.5 (O1); no longer U46.~ (Oin)
- net Q5SR: now also SPE8.2 (Set/Reset); no longer SPE8.~ (Set/Reset)
- net Q5V: now also U47.5 (O1); no longer U47.~ (Oin)
- net Q6H: now also U48.5 (O1); no longer U48.~ (Oin)
- net Q6SR: now also SPE6.2 (Set/Reset); no longer SPE6.~ (Set/Reset)
- net Q6V: now also U49.5 (O1); no longer U49.~ (Oin)
- net Q7H: now also U50.5 (O1); no longer U50.~ (Oin)
- net Q7SR: now also SPE4.2 (Set/Reset); no longer SPE4.~ (Set/Reset)
- net Q7V: now also U51.5 (O1); no longer U51.~ (Oin)
- net Q8H: now also U71.5 (O1); no longer U71.~ (Oin)
- net Q8SR: now also SPE2.2 (Set/Reset); no longer SPE2.~ (Set/Reset)
- net Q8V: now also U72.5 (O1); no longer U72.~ (Oin)
- net VCC: now also CH1.10 (Vcc), CX1.10 (Vcc), CY1.10 (Vcc), CZ1.10 (Vcc), SPE1.8 (Vcc), SPE2.8 (Vcc), SPE3.8 (Vcc), SPE4.8 (Vcc), SPE5.8 (Vcc), SPE6.8 (Vcc), SPE7.8 (Vcc), SPE8.8 (Vcc); no longer CH1.~ (Vcc), CX1.~ (Vcc), CY1.~ (Vcc), CZ1.~ (Vcc), SPE1.7 (Vcc), SPE2.7 (Vcc), SPE3.7 (Vcc), SPE4.7 (Vcc), SPE5.7 (Vcc), SPE6.7 (Vcc), SPE7.7 (Vcc), SPE8.7 (Vcc)
- net VSS: now also CH1.9 (GND), CX1.9 (GND), CY1.9 (GND), CZ1.9 (GND); no longer CH1.~ (Vcc), CX1.~ (Vcc), CY1.~ (Vcc), CZ1.~ (Vcc)
- net at X8.3 (Vout): now also U28.4 (S4); no longer U28.~ (S5)
- net at X8.4 (Hout): now also U43.4 (S4); no longer U43.~ (S5)
- net at Y8.3 (Vout): now also U28.3 (S3); no longer U28.~ (S5)
- net at Y8.4 (Hout): now also U43.3 (S3); no longer U43.~ (S5)
- net at Z8.3 (Vout): now also U28.2 (S2); no longer U28.~ (S5)
- net at Z8.4 (Hout): now also U43.2 (S2); no longer U43.~ (S5)
- net at CZ1.5 (V-out): now also U154.3 (S3); no longer U154.~ (S5)
- net at CZ1.6 (H-out): now also U164.3 (S3); no longer U164.~ (S5)
- net at CZ1.7 (V-out): now also U153.2 (S2); no longer U153.~ (S5)
- net at CZ1.8 (H-out): now also U163.2 (S2); no longer U163.~ (S5)
- net at H8.3 (Vout): now also U28.1 (S1); no longer U28.~ (S5)
- net at H8.4 (Hout): now also U43.1 (S1); no longer U43.~ (S5)
- net at CX1.5 (V-out): now also U154.1 (S1); no longer U154.~ (S5)
- net at CX1.6 (H-out): now also U164.1 (S1); no longer U164.~ (S5)
- net at CX1.7 (V-out): now also U153.4 (S4); no longer U153.~ (S5)
- net at CX1.8 (H-out): now also U163.4 (S4); no longer U163.~ (S5)
- net at CY1.5 (V-out): now also U154.4 (S4); no longer U154.~ (S5)
- net at CY1.6 (H-out): now also U164.4 (S4); no longer U164.~ (S5)
- net at CY1.7 (V-out): now also U153.1 (S1); no longer U153.~ (S5)
- net at CY1.8 (H-out): now also U163.1 (S1); no longer U163.~ (S5)
- net at SPE1.4 (GND): no longer U83.~ (S5)
- net at SPE1.5 (H): now also U83.3 (S3); no longer U82.~ (S5)
- net at X6.3 (Vout): now also U56.4 (S4); no longer U56.~ (S5)
- net at X6.4 (Hout): now also U77.4 (S4); no longer U77.~ (S5)
- net at Y6.3 (Vout): now also U56.3 (S3); no longer U56.~ (S5)
- net at Y6.4 (Hout): now also U77.3 (S3); no longer U77.~ (S5)
- net at Z6.3 (Vout): now also U56.2 (S2); no longer U56.~ (S5)
- net at Z6.4 (Hout): now also U77.2 (S2); no longer U77.~ (S5)
- net at H6.3 (Vout): now also U56.1 (S1); no longer U56.~ (S5)
- net at H6.4 (Hout): now also U77.1 (S1); no longer U77.~ (S5)
- net at CH1.5 (V-out): now also U154.2 (S2); no longer U154.~ (S5)
- net at CH1.6 (H-out): now also U164.2 (S2); no longer U164.~ (S5)
- net at CH1.7 (V-out): now also U153.3 (S3); no longer U153.~ (S5)
- net at CH1.8 (H-out): now also U163.3 (S3); no longer U163.~ (S5)
- net at U34.~ (Oin): now also U28.6 (Out); no longer U40.~ (Oin)
- net at U45.~ (Oin): now also U43.6 (Out); no longer U53.~ (Oin)
- net at U68.~ (Oin): now also U56.6 (Out); no longer U74.~ (Oin)
- net at U85.~ (Oin): now also U77.6 (Out); no longer U91.~ (Oin)
- net at U102.~ (Oin): now also U96.6 (Out); no longer U106.~ (Oin)
- net at X4.3 (Vout): now also U96.4 (S4); no longer U96.~ (S5)
- net at Y4.3 (Vout): now also U96.3 (S3); no longer U96.~ (S5)
- net at Z4.3 (Vout): now also U96.2 (S2); no longer U96.~ (S5)
- net at H4.3 (Vout): now also U96.1 (S1); no longer U96.~ (S5)
- net at U118.~ (Oin): now also U114.6 (Out); no longer U124.~ (Oin)
- net at X4.4 (Hout): now also U114.4 (S4); no longer U114.~ (S5)
- net at Y4.4 (Hout): now also U114.3 (S3); no longer U114.~ (S5)
- net at Z4.4 (Hout): now also U114.2 (S2); no longer U114.~ (S5)
- net at H4.4 (Hout): now also U114.1 (S1); no longer U114.~ (S5)
- net at X2.3 (Vout): now also U128.4 (S4); no longer U128.~ (S5)
- net at X2.4 (Hout): now also U144.4 (S4); no longer U144.~ (S5)
- net at Y2.3 (Vout): now also U128.3 (S3); no longer U128.~ (S5)
- net at Y2.4 (Hout): now also U144.3 (S3); no longer U144.~ (S5)
- net at Z2.3 (Vout): now also U128.2 (S2); no longer U128.~ (S5)
- net at Z2.4 (Hout): now also U144.2 (S2); no longer U144.~ (S5)
- net at H2.3 (Vout): now also U128.1 (S1); no longer U128.~ (S5)
- net at H2.4 (Hout): now also U144.1 (S1); no longer U144.~ (S5)
- net at U130.~ (Oin): now also U128.6 (Out); no longer U136.~ (Oin)
- net at U146.~ (Oin): now also U144.6 (Out); no longer U148.~ (Oin)
- net at U158.~ (Oin): now also U154.6 (Out); no longer U160.~ (Oin)
- net at U166.~ (Oin): now also U164.6 (Out); no longer U168.~ (Oin)
- net at SPE3.4 (GND): no longer U104.~ (S2)
- net at SPE3.5 (H): now also U104.2 (S2); no longer U103.~ (S2)
- net at SPE5.4 (GND): no longer U132.~ (S2)
- net at SPE5.5 (H): now also U132.2 (S2); no longer U131.~ (S2)
- net at SPE7.4 (GND): no longer U150.~ (S2)
- net at SPE7.5 (H): now also U150.2 (S2); no longer U149.~ (S2)
- net at SPE8.4 (GND): no longer U156.~ (S2)
- net at SPE8.5 (H): now also U156.2 (S2); no longer U155.~ (S2)
- net at X7.3 (Vout): now also U27.4 (S4); no longer U27.~ (S5)
- net at X7.4 (Hout): now also U42.4 (S4); no longer U42.~ (S5)
- net at Y7.3 (Vout): now also U27.3 (S3); no longer U27.~ (S5)
- net at Y7.4 (Hout): now also U42.3 (S3); no longer U42.~ (S5)
- net at Z7.3 (Vout): now also U27.2 (S2); no longer U27.~ (S5)
- net at Z7.4 (Hout): now also U42.2 (S2); no longer U42.~ (S5)
- net at H7.3 (Vout): now also U27.1 (S1); no longer U27.~ (S5)
- net at H7.4 (Hout): now also U42.1 (S1); no longer U42.~ (S5)
- net at X5.3 (Vout): now also U55.4 (S4); no longer U55.~ (S5)
- net at X5.4 (Hout): now also U76.4 (S4); no longer U76.~ (S5)
- net at Y5.3 (Vout): now also U55.3 (S3); no longer U55.~ (S5)
- net at Y5.4 (Hout): now also U76.3 (S3); no longer U76.~ (S5)
- net at Z5.3 (Vout): now also U55.2 (S2); no longer U55.~ (S5)
- net at Z5.4 (Hout): now also U76.2 (S2); no longer U76.~ (S5)
- net at H5.3 (Vout): now also U55.1 (S1); no longer U55.~ (S5)
- net at H5.4 (Hout): now also U76.1 (S1); no longer U76.~ (S5)
- net at U33.~ (Oin): now also U27.6 (Out); no longer U39.~ (Oin)
- net at U44.~ (Oin): now also U42.6 (Out); no longer U52.~ (Oin)
- net at U67.~ (Oin): now also U55.6 (Out); no longer U73.~ (Oin)
- net at U84.~ (Oin): now also U76.6 (Out); no longer U90.~ (Oin)
- net at U101.~ (Oin): now also U95.6 (Out); no longer U105.~ (Oin)
- net at X3.3 (Vout): now also U95.4 (S4); no longer U95.~ (S5)
- net at Y3.3 (Vout): now also U95.3 (S3); no longer U95.~ (S5)
- net at Z3.3 (Vout): now also U95.2 (S2); no longer U95.~ (S5)
- net at H3.3 (Vout): now also U95.1 (S1); no longer U95.~ (S5)
- net at U117.~ (Oin): now also U113.6 (Out); no longer U123.~ (Oin)
- net at X3.4 (Hout): now also U113.4 (S4); no longer U113.~ (S5)
- net at Y3.4 (Hout): now also U113.3 (S3); no longer U113.~ (S5)
- net at Z3.4 (Hout): now also U113.2 (S2); no longer U113.~ (S5)
- net at H3.4 (Hout): now also U113.1 (S1); no longer U113.~ (S5)
- net at X1.3 (Vout): now also U127.4 (S4); no longer U127.~ (S5)
- net at X1.4 (Hout): now also U143.4 (S4); no longer U143.~ (S5)
- net at Y1.3 (Vout): now also U127.3 (S3); no longer U127.~ (S5)
- net at Y1.4 (Hout): now also U143.3 (S3); no longer U143.~ (S5)
- net at Z1.3 (Vout): now also U127.2 (S2); no longer U127.~ (S5)
- net at Z1.4 (Hout): now also U143.2 (S2); no longer U143.~ (S5)
- net at H1.3 (Vout): now also U127.1 (S1); no longer U127.~ (S5)
- net at H1.4 (Hout): now also U143.1 (S1); no longer U143.~ (S5)
- net at U129.~ (Oin): now also U127.6 (Out); no longer U135.~ (Oin)
- net at U145.~ (Oin): now also U143.6 (Out); no longer U147.~ (Oin)
- net at U157.~ (Oin): now also U153.6 (Out); no longer U159.~ (Oin)
- net at U165.~ (Oin): now also U163.6 (Out); no longer U167.~ (Oin)
- net at SPE6.4 (GND): no longer U139.~ (S2)
- net at SPE6.5 (H): now also U139.2 (S2); no longer U138.~ (S2)
- net at SPE4.4 (GND): no longer U120.~ (S2)
- net at SPE4.5 (H): now also U120.2 (S2); no longer U119.~ (S2)
- net at SPE2.4 (GND): no longer U94.~ (S5)
- net at SPE2.5 (H): now also U94.5 (S5); no longer U93.~ (S5)
- new net: M8.5 (H), U38.5 (O1)
- new net: M8.6 (V), U37.5 (O1)
- new net: SPE1.6 (V), U82.3 (S3)
- new net: U25.~ (Vcc), U37.4 (O2)
- new net: U37.6 (Oin), U57.4 (O2)
- new net: U25.~ (Vcc), U26.~ (Vcc)
- new net: U26.~ (Vcc), U38.4 (O2)
- new net: U28.5 (S5), U40.4 (O2)
- new net: U40.5 (O1), U82.5 (S5)
- new net: U34.~ (Oin), U40.6 (Oin)
- new net: U45.~ (Oin), U53.6 (Oin)
- new net: U43.5 (S5), U53.4 (O2)
- new net: U53.5 (O1), U83.4 (S4)
- new net: U56.5 (S5), U74.4 (O2)
- new net: U74.5 (O1), U87.2 (S2)
- new net: U68.~ (Oin), U74.6 (Oin)
- new net: U85.~ (Oin), U91.6 (Oin)
- new net: U77.5 (S5), U91.4 (O2)
- new net: U89.2 (S2), U91.5 (O1)
- new net: U106.4 (O2), U96.5 (S5)
- new net: U106.5 (O1), U112.6 (Oin)
- new net: U102.~ (Oin), U106.6 (Oin)
- new net: U118.~ (Oin), U124.6 (Oin)
- new net: U114.5 (S5), U124.4 (O2)
- new net: U124.5 (O1), U126.6 (Oin)
- new net: U38.6 (Oin), U58.4 (O2)
- new net: U112.4 (O2), U116.2 (S2)
- new net: U122.2 (S2), U126.4 (O2)
- new net: U128.5 (S5), U136.4 (O2)
- new net: U136.5 (O1), U141.6 (Oin)
- new net: U130.~ (Oin), U136.6 (Oin)
- new net: U146.~ (Oin), U148.6 (Oin)
- new net: U144.5 (S5), U148.4 (O2)
- new net: U148.5 (O1), U152.6 (Oin)
- new net: U134.2 (S2), U141.4 (O2)
- new net: U154.5 (S5), U160.4 (O2)
- new net: U160.5 (O1), U162.6 (Oin)
- new net: U158.~ (Oin), U160.6 (Oin)
- new net: U166.~ (Oin), U168.6 (Oin)
- new net: U164.5 (S5), U168.4 (O2)
- new net: U168.5 (O1), U170.6 (Oin)
- new net: U162.4 (O2), U173.~ (Vcc)
- new net: U170.4 (O2), U174.~ (Vcc)
- new net: U31.6 (Oin), U63.4 (O2)
- new net: U63.6 (Oin), U87.3 (Out)
- new net: U32.6 (Oin), U64.4 (O2)
- new net: U64.6 (Oin), U89.3 (Out)
- new net: M6.5 (H), U32.5 (O1)
- new net: M6.6 (V), U31.5 (O1)
- new net: U17.~ (Vcc), U31.4 (O2)
- new net: U17.~ (Vcc), U18.~ (Vcc)
- new net: U18.~ (Vcc), U32.4 (O2)
- new net: M4.5 (H), U22.5 (O1)
- new net: M4.6 (V), U21.5 (O1)
- new net: U21.4 (O2), U9.~ (Vcc)
- new net: U21.6 (Oin), U65.4 (O2)
- new net: U10.~ (Vcc), U9.~ (Vcc)
- new net: U10.~ (Vcc), U22.4 (O2)
- new net: U22.6 (Oin), U66.4 (O2)
- new net: M2.5 (H), U14.5 (O1)
- new net: M2.6 (V), U13.5 (O1)
- new net: U13.4 (O2), U5.~ (Vcc)
- new net: U13.6 (Oin), U69.4 (O2)
- new net: U5.~ (Vcc), U6.~ (Vcc)
- new net: U14.4 (O2), U6.~ (Vcc)
- new net: U14.6 (Oin), U70.4 (O2)
- new net: SPE3.6 (V), U103.1 (S1)
- new net: U104.1 (S1), U174.~ (Vcc)
- new net: U104.3 (Out), U89.1 (S1)
- new net: U103.2 (S2), U173.~ (Vcc)
- new net: U103.3 (Out), U87.1 (S1)
- new net: U59.~ (Vcc), U78.3 (Out)
- new net: U60.~ (Vcc), U79.3 (Out)
- new net: U61.~ (Vcc), U80.3 (Out)
- new net: U62.~ (Vcc), U81.3 (Out)
- new net: SPE5.6 (V), U131.1 (S1)
- new net: U132.1 (S1), U174.~ (Vcc)
- new net: U122.1 (S1), U132.3 (Out)
- new net: U131.2 (S2), U173.~ (Vcc)
- new net: U116.1 (S1), U131.3 (Out)
- new net: U116.3 (Out), U65.6 (Oin)
- new net: U122.3 (Out), U66.6 (Oin)
- new net: U78.2 (S2), U97.4 (O2)
- new net: U80.2 (S2), U97.5 (O1)
- new net: U107.6 (Out), U97.6 (Oin)
- new net: SPE7.6 (V), U149.1 (S1)
- new net: U142.1 (S1), U150.3 (Out)
- new net: U149.2 (S2), U173.~ (Vcc)
- new net: U134.1 (S1), U149.3 (Out)
- new net: U79.2 (S2), U98.4 (O2)
- new net: U80.1 (S1), U98.5 (O1)
- new net: U108.6 (Out), U98.6 (Oin)
- new net: U100.4 (O2), U81.1 (S1)
- new net: U100.5 (O1), U79.1 (S1)
- new net: U100.6 (Oin), U110.6 (Out)
- new net: U81.2 (S2), U99.4 (O2)
- new net: U78.1 (S1), U99.5 (O1)
- new net: U109.6 (Out), U99.6 (Oin)
- new net: U142.3 (Out), U70.6 (Oin)
- new net: U134.3 (Out), U69.6 (Oin)
- new net: U173.~ (Vcc), U82.4 (S4)
- new net: U174.~ (Vcc), U83.2 (S2)
- new net: SPE8.6 (V), U155.1 (S1)
- new net: U156.1 (S1), U172.~ (Vcc)
- new net: U133.1 (S1), U156.3 (Out)
- new net: U155.2 (S2), U171.~ (Vcc)
- new net: U137.1 (S1), U155.3 (Out)
- new net: M7.5 (H), U35.5 (O1)
- new net: M7.6 (V), U36.5 (O1)
- new net: U24.~ (Vcc), U36.4 (O2)
- new net: U36.6 (Oin), U72.4 (O2)
- new net: U23.~ (Vcc), U24.~ (Vcc)
- new net: U23.~ (Vcc), U35.4 (O2)
- new net: U27.5 (S5), U39.4 (O2)
- new net: U39.5 (O1), U41.6 (Oin)
- new net: U33.~ (Oin), U39.6 (Oin)
- new net: U44.~ (Oin), U52.6 (Oin)
- new net: U42.5 (S5), U52.4 (O2)
- new net: U52.5 (O1), U54.6 (Oin)
- new net: U55.5 (S5), U73.4 (O2)
- new net: U73.5 (O1), U75.6 (Oin)
- new net: U67.~ (Oin), U73.6 (Oin)
- new net: U84.~ (Oin), U90.6 (Oin)
- new net: U76.5 (S5), U90.4 (O2)
- new net: U90.5 (O1), U92.6 (Oin)
- new net: U105.4 (O2), U95.5 (S5)
- new net: U105.5 (O1), U111.6 (Oin)
- new net: U101.~ (Oin), U105.6 (Oin)
- new net: U117.~ (Oin), U123.6 (Oin)
- new net: U113.5 (S5), U123.4 (O2)
- new net: U123.5 (O1), U125.6 (Oin)
- new net: U35.6 (Oin), U71.4 (O2)
- new net: U54.4 (O2), U93.3 (S3)
- new net: U41.4 (O2), U94.3 (S3)
- new net: U75.4 (O2), U86.2 (S2)
- new net: U88.2 (S2), U92.4 (O2)
- new net: U111.4 (O2), U115.2 (S2)
- new net: U121.2 (S2), U125.4 (O2)
- new net: U127.5 (S5), U135.4 (O2)
- new net: U135.5 (O1), U140.6 (Oin)
- new net: U129.~ (Oin), U135.6 (Oin)
- new net: U145.~ (Oin), U147.6 (Oin)
- new net: U143.5 (S5), U147.4 (O2)
- new net: U147.5 (O1), U151.6 (Oin)
- new net: U133.2 (S2), U140.4 (O2)
- new net: U137.2 (S2), U151.4 (O2)
- new net: U153.5 (S5), U159.4 (O2)
- new net: U159.5 (O1), U161.6 (Oin)
- new net: U157.~ (Oin), U159.6 (Oin)
- new net: U165.~ (Oin), U167.6 (Oin)
- new net: U163.5 (S5), U167.4 (O2)
- new net: U167.5 (O1), U169.6 (Oin)
- new net: U161.4 (O2), U172.~ (Vcc)
- new net: U169.4 (O2), U171.~ (Vcc)
- new net: M5.5 (H), U29.5 (O1)
- new net: M5.6 (V), U30.5 (O1)
- new net: U16.~ (Vcc), U30.4 (O2)
- new net: U30.6 (Oin), U51.4 (O2)
- new net: U15.~ (Vcc), U16.~ (Vcc)
- new net: U15.~ (Vcc), U29.4 (O2)
- new net: U29.6 (Oin), U50.4 (O2)
- new net: M3.5 (H), U19.5 (O1)
- new net: M3.6 (V), U20.5 (O1)
- new net: U20.4 (O2), U8.~ (Vcc)
- new net: U20.6 (Oin), U49.4 (O2)
- new net: U7.~ (Vcc), U8.~ (Vcc)
- new net: U19.4 (O2), U7.~ (Vcc)
- new net: U19.6 (Oin), U48.4 (O2)
- new net: M1.5 (H), U11.5 (O1)
- new net: M1.6 (V), U12.5 (O1)
- new net: U12.4 (O2), U4.~ (Vcc)
- new net: U12.6 (Oin), U47.4 (O2)
- new net: U3.~ (Vcc), U4.~ (Vcc)
- new net: U11.4 (O2), U3.~ (Vcc)
- new net: U11.6 (Oin), U46.4 (O2)
- new net: U119.3 (Out), U88.1 (S1)
- new net: U50.6 (Oin), U88.3 (Out)
- new net: U120.3 (Out), U86.1 (S1)
- new net: U51.6 (Oin), U86.3 (Out)
- new net: U121.1 (S1), U138.3 (Out)
- new net: U121.3 (Out), U48.6 (Oin)
- new net: U115.1 (S1), U139.3 (Out)
- new net: U115.3 (Out), U49.6 (Oin)
- new net: U137.3 (Out), U46.6 (Oin)
- new net: U133.3 (Out), U47.6 (Oin)
- new net: U171.~ (Vcc), U172.~ (Vcc)
- new net: U139.1 (S1), U172.~ (Vcc)
- new net: U120.1 (S1), U172.~ (Vcc)
- new net: U172.~ (Vcc), U94.4 (S4)
- new net: U138.2 (S2), U171.~ (Vcc)
- new net: U119.2 (S2), U171.~ (Vcc)
- new net: U171.~ (Vcc), U93.5 (S5)
- new net: SPE6.6 (V), U138.1 (S1)
- new net: SPE4.6 (V), U119.1 (S1)
- new net: SPE2.6 (V), U93.4 (S4)
- new net: U71.6 (Oin), U93.6 (Out)
- new net: U72.6 (Oin), U94.6 (Out)
- new net: U57.6 (Oin), U82.6 (Out)
- new net: U58.6 (Oin), U83.6 (Out)
